File: console/console.kicad_pcb (KiCad board)
At the start: 2 copper layers, 15 parts

Commit message: PCB complete, not tested yet
Parts:
- ARDUINO1: moved to B.Cu
- SW_Left1, SW_Right1: footprint footprints custom 1:D6R90F2LFS -> digikey-footprints:D6R90F2LFS
- SW_Left_Table_Control1, SW_Right_Table_Control1, SW_Selector1: footprint footprints custom 2:XDCR_PEC11R-4215F-S0024 -> digikey-footprints:XDCR_PEC11R-4215F-S0024
- moved RV_Left_Bass1 177.0 mm to (80.0, 171.4), turned to 270 degrees
- moved SW_Selector1 154.5 mm to (114.3, 180.3)
- moved RV_Left_Treble1 132.1 mm to (80.0, 134.6), turned to 270 degrees
- moved RV_Right_Mid2 129.4 mm to (80.0, 153.7), turned to 270 degrees
- moved SW_Left_Table_Control1 124.2 mm to (61.0, 109.2)
- moved RV_Right_BPM1 110.4 mm to (166.4, 25.4), turned to 270 degrees
- moved RV_Left_BPM1 105.5 mm to (63.1, 25.4), turned to 270 degrees
- moved SW_Left1 92.7 mm to (78.8, 120.7)
- moved SW_Right1 91.9 mm to (142.5, 120.7)
- moved RV_Right_Bass1 87.2 mm to (141.0, 171.4), turned to 270 degrees
- moved RV_Left_Mid1 83.9 mm to (141.0, 153.7), turned to 270 degrees
- moved RV_Crossfader1 69.7 mm to (76.5, 106.7)
- moved RV_Right_Treble1 62.9 mm to (141.0, 135.9), turned to 270 degrees
- moved SW_Right_Table_Control1 59.2 mm to (165.1, 109.2)
- moved ARDUINO1 34.3 mm to (88.9, 48.3), turned to 270 degrees
- renumbered RV_Left_Mid2 to RV_Right_Mid2
Connections:
- RV_Crossfader1 pad 1: Net-(ARDUINO1-Pad5) -> Net-(ARDUINO1-Pad7)
- RV_Crossfader1 pad 2: Net-(RV_Crossfader1-Pad2) -> Net-(ARDUINO1-Pad9)
- RV_Crossfader1 pad 3: Net-(ARDUINO1-Pad7) -> Net-(ARDUINO1-Pad5)
Routing:
- net Net-(ARDUINO1-Pad5): track 0.00 -> 597.2 mm, vias 0 -> 2
- net Net-(ARDUINO1-Pad7): track 0.00 -> 397.7 mm
- net Net-(ARDUINO1-Pad13): track 0.00 -> 142.5 mm
- net Net-(ARDUINO1-Pad28): track 0.00 -> 139.0 mm
- net Net-(ARDUINO1-Pad22): track 0.00 -> 131.6 mm, vias 0 -> 3
- net Net-(ARDUINO1-Pad25): track 0.00 -> 126.6 mm
- net Net-(ARDUINO1-Pad21): track 0.00 -> 126.2 mm, vias 0 -> 3
- net Net-(ARDUINO1-Pad15): track 0.00 -> 119.8 mm, vias 0 -> 1
- net Net-(ARDUINO1-Pad16): track 0.00 -> 118.1 mm, vias 0 -> 2
- net Net-(ARDUINO1-Pad11): track 0.00 -> 118.1 mm
- net Net-(ARDUINO1-Pad17): track 0.00 -> 117.0 mm, vias 0 -> 3
- net Net-(ARDUINO1-Pad12): track 0.00 -> 113.7 mm, vias 0 -> 1
- net Net-(ARDUINO1-Pad19): track 0.00 -> 102.1 mm, vias 0 -> 3
- net Net-(ARDUINO1-Pad23): track 0.00 -> 101.2 mm, vias 0 -> 3
- net Net-(ARDUINO1-Pad26): track 0.00 -> 100.9 mm
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
Commit message: added edges
Parts:
- moved ARDUINO1 19.1 mm to (69.8, 48.3)
- moved RV_Right_BPM1 19.1 mm to (147.4, 25.4)
- moved RV_Crossfader1 19.1 mm to (57.5, 106.7)
- moved RV_Left_Bass1 19.1 mm to (61.0, 171.4)
- moved RV_Left_Treble1 19.1 mm to (61.0, 134.6)
- moved RV_Right_Mid2 19.1 mm to (61.0, 153.7)
- moved SW_Left_Table_Control1 19.1 mm to (41.9, 109.2)
- moved RV_Left_BPM1 19.0 mm to (44.1, 25.4)
- moved RV_Left_Mid1 19.0 mm to (121.9, 153.7)
- moved RV_Right_Bass1 19.0 mm to (121.9, 171.4)
- moved RV_Right_Treble1 19.0 mm to (121.9, 135.9)
- moved SW_Left1 19.0 mm to (59.8, 120.7)
- moved SW_Right1 19.0 mm to (123.4, 120.7)
- moved SW_Selector1 19.0 mm to (95.2, 180.3)
- moved SW_Right_Table_Control1 19.0 mm to (146.1, 109.2)
Other:
- board outline added: 141 x 181.6 mm
- board text added: "Designed by Oloturia v.1.0 26-Jan-2024"

Commit message: error corrected, gerber files created
Routing:
- net Net-(ARDUINO1-Pad5): track 597.2 -> 565.4 mm
- net Net-(ARDUINO1-Pad9): track 47.2 -> 47.9 mm
Changed lines of the file:
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@@
     (thickness 1.6)
     (drawings 5)
-    (tracks 280)
+    (tracks 278)
     (zones 0)
     (modules 15)
@@
       (psnegative false)
       (psa4output false)
-      (plotreference true)
-      (plotvalue true)
+      (plotreference false)
+      (plotvalue false)
       (plotinvisibletext false)
       (padsonsilk false)
@@
       (outputformat 1)
       (mirror false)
-      (drillshape 1)
+      (drillshape 0)
       (scaleselection 1)
-      (outputdirectory ""))
+      (outputdirectory "./"))
   )
   (net 0 "")
@@
   (segment (start 64.77 71.12) (end 62.23 73.66) (width 0.25) (layer F.Cu) (net 14))
   (segment (start 62.23 73.66) (end 62.23 76.2) (width 0.25) (layer F.Cu) (net 14))
-  (segment (start 62.23 76.2) (end 59.69 78.74) (width 0.25) (layer B.Cu) (net 14))
-  (segment (start 59.69 107.95) (end 57.46 110.18) (width 0.25) (layer B.Cu) (net 14))
-  (segment (start 59.69 78.74) (end 59.69 107.95) (width 0.25) (layer B.Cu) (net 14))
+  (segment (start 59.69 78.74) (end 62.23 76.2) (width 0.25) (layer B.Cu) (net 14))
+  (segment (start 59.69 109.22) (end 59.69 78.74) (width 0.25) (layer B.Cu) (net 14))
+  (segment (start 58.73 110.18) (end 59.69 109.22) (width 0.25) (layer B.Cu) (net 14))
+  (segment (start 57.46 110.18) (end 58.73 110.18) (width 0.25) (layer B.Cu) (net 14))
   (segment (start 143.55 102.22) (end 143.55 91.48) (width 0.25) (layer B.Cu) (net 15))
   (segment (start 143.55 91.48) (end 130.81 78.74) (width 0.25) (layer B.Cu) (net 15))
@@
   (segment (start 55.88 148.59) (end 55.88 139.7) (width 0.25) (layer F.Cu) (net 22))
   (segment (start 55.88 139.7) (end 60.96 134.62) (width 0.25) (layer F.Cu) (net 22))
-  (segment (start 57.46 106.68) (end 54.61 109.53) (width 0.25) (layer B.Cu) (net 22))
-  (segment (start 54.61 128.27) (end 60.96 134.62) (width 0.25) (layer B.Cu) (net 22))
-  (segment (start 54.61 109.53) (end 54.61 128.27) (width 0.25) (layer B.Cu) (net 22))
   (segment (start 133.130501 177.580501) (end 127 183.711002) (width 0.25) (layer F.Cu) (net 22))
   (via (at 133.130501 177.580501) (size 0.8) (drill 0.4) (layers F.Cu B.Cu) (net 22))

Commit message: corrected small error
Routing:
- net Net-(ARDUINO1-Pad19): track 102.1 -> 101.4 mm
Changed lines of the file:
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@@
     (thickness 1.6)
     (drawings 5)
-    (tracks 278)
+    (tracks 279)
     (zones 0)
     (modules 15)
@@
     (visible_elements FFFFFF7F)
     (pcbplotparams
-      (layerselection 0x010fc_ffffffff)
+      (layerselection 0x00000_7fffffff)
       (usegerberextensions false)
       (usegerberattributes false)
@@
   (segment (start 44.41 116.72) (end 50.92 116.72) (width 0.25) (layer F.Cu) (net 25))
   (segment (start 50.92 116.72) (end 53.34 114.3) (width 0.25) (layer F.Cu) (net 25))
-  (segment (start 53.34 114.3) (end 53.34 102.87) (width 0.25) (layer F.Cu) (net 25))
   (segment (start 61.690998 102.87) (end 62.960998 101.6) (width 0.25) (layer F.Cu) (net 25))
-  (segment (start 53.34 102.87) (end 61.690998 102.87) (width 0.25) (layer F.Cu) (net 25))
   (segment (start 62.960998 101.6) (end 82.55 101.6) (width 0.25) (layer F.Cu) (net 25))
   (via (at 104.14 80.01) (size 0.8) (drill 0.4) (layers F.Cu B.Cu) (net 25))
@@
   (segment (start 113.03 69.85) (end 114.3 69.85) (width 0.25) (layer B.Cu) (net 25))
   (segment (start 114.3 69.85) (end 118.11 73.66) (width 0.25) (layer B.Cu) (net 25))
+  (segment (start 53.34 114.3) (end 53.34 104.14) (width 0.25) (layer F.Cu) (net 25))
+  (segment (start 53.34 104.14) (end 54.61 102.87) (width 0.25) (layer F.Cu) (net 25))
+  (segment (start 54.61 102.87) (end 61.690998 102.87) (width 0.25) (layer F.Cu) (net 25))
   (segment (start 127 80.01) (end 127 77.47) (width 0.25) (layer B.Cu) (net 27))
   (segment (start 143.55 116.72) (end 139.58 116.72) (width 0.25) (layer B.Cu) (net 27))

Commit message: updated kicad version, added gitignore
Other:
- net class Default removed
